Commit message: feat(s6): 실차 S6 인수 준비물 6종 완료 — 예약 19 코드 반영 + 런북·검증 도구 4종
인수일(08-03) 하루 전, 로봇 없이 만들 수 있는 것을 전부 만들었다.

## S6-7 = 예약 19 (src/tunnel_bringup/** 동결 예외 4회차)

② Nav2 속도 상한 [0.30,0,0.80] → [0.12,0,0.50] (min_velocity 도 함께 — 경계는 양쪽)
③ URDF base_footprint→base_link z 0.065 → 0.053 (하중 상태 실측 축높이)
④ URDF imu_link xyz="0 0 0.339" rpy="0 0 -1.5708" (바닥기준 392mm − 축높이 53mm)
⑤ serial_baud 921600 → 115200 (런치 2파일) · ekf 주기 주석 46.4Hz/20~23ms

★ ①(EKF QoS)은 코드 변경 없음 — 전제가 실측으로 뒤집혔다:
  ⓐ robot_localization 3.5.4 의 /odom·/imu/data 구독은 **이미 BEST_EFFORT**
  ⓑ 구독 QoS 오버라이드 파라미터가 **존재하지 않는다** (qos_overrides 는 퍼블리셔 3개뿐)
  → 계획대로 yaml 한 줄을 넣었다면 무시된 채 "막았다"는 기록만 남았을 것이다.
  조치 대신 **검사**로 닫았다 (d0_check.sh 가 토픽 전체를 훑는다).

같은 클래스 전수: /odom 구독자 3종(ekf·bt_navigator·controller_server) 전부 BEST_EFFORT,
velocity_smoother 는 구독 자체를 안 함(OPEN_LOOP), /imu/data 는 EKF 하나. /scan 은 발행자가
RELIABLE 이라 무관. → 위험은 '아는 목록'에 없어 목록 대신 검사로 닫았다.

관측으로 확인 (주장 아님): tf2_echo base_footprint→imu_link = 0.392 m · yaw −90°
(구동부 바닥기준 실측과 일치 — 기준면 뺄셈이 왕복으로 닫혔다), →base_link = 0.053.

경계: tunnel_sim · mission_manager · 노드 코드 · test/ diff 0 (gate_fakes.py 무변경).

## S6-1~S6-5 (tools/ · docs/)

- docs/JETSON_SETUP.md — 셋업 런북 + micro_ros_agent 확보 2안(S6-2)
  apt 부재를 대조군과 함께 확인 · Docker 이미지 linux/arm64 지원을 manifest 로 확인
- docs/D1_FIRST_STEP.md — D+1 첫 스텝(agent→라이다 장착·측정→TF→EKF→R3 rosbag 분석)
- tools/d0_check.sh — D+0 판정 6검사. 가짜 ros2 로 10 시나리오 실행 검증,
  종료 0/1/2(불완전) 계약 확인. scan_unbounded_cli 0건 · bash -n 통과
- tools/bag_gap_report.py — R3 간격 분포. 실제 녹화 bag 으로 검증(549개·46.50Hz·max 24.39ms)
- tools/udev/99-teensy-drive.rules — VID/PID 는 TODO(D+0) + 확인 명령까지

★ 새 D+0 즉발 함정 발견: sllidar_ros2 가 저장소에 없다(.gitignore, 추적 0건). 그런데
tunnel_bringup/package.xml 이 의존으로 선언 → 새로 clone 한 Jetson 에서 빌드 실패.
MASTER_PLAN §3 포터빌리티 표의 "clone 불필요 ✅" 는 노트북 기준이었다 — 정정했다.

## 회귀

pytest 182 · colcon 245(0e·0f·3s) · doc_check --strict 전항목 OK.
test_gate_regression 14/14 — 참고 기록이며 판정 근거로 쓰지 않았다(§24.5a flake 미규명).

## 공개하는 잔여 위험

- 속도 상한을 펌웨어 값으로 내리자 desired_linear_vel(0.12)·rotate_to_heading(0.5)이
  상한과 같아졌다 → 곡선에서 잘릴 수 있고 잘림은 Nav2 에 보고되지 않는다. R6 판정 항목.
- d0_check·bag_gap_report 판정 논리는 세션 검증만 있고 저장소 회귀가 아니다 → 예약 21.
- agent 확보 2안 모두 Jetson 네트워크가 필요하다.

문서: MASTER_PLAN §3/§7(예약 19 종결·예약 21 신설) · FREEZE_MANIFEST §10.4.1 ·
REAL_ROBOT_VALUES §1-b/§2/§5 · CURRENT_HANDOFF → 실차 D+0 · 0801_현황 §20.

Co-Authored-By: Claude Opus 5 (1M context) <noreply@anthropic.com>
Claude-Session: https://claude.ai/code/session_01DRyuoA8Mgc5RK9baWBGvjK

File: src/tunnel_bringup/urdf/robot_real.urdf (robot description, URDF)
Before this commit: robot tunnel_robot_real, 6 links, 5 joints
Joints:
- joint base_joint: origin xyz=0 0 0.065 rpy=0 0 0 -> xyz=0 0 0.053 rpy=0 0 0
- joint imu_joint: origin xyz=0 0 0 rpy=0 0 0 -> xyz=0 0 0.339 rpy=0 0 -1.5708

Commit message: urdf(lidar): a placeholder zero that survives the measurement writes a silently wrong map
`lidar_joint origin` 은 `xyz="0 0 0"` 이었다. 그 0 은 값이 아니라 파일 주석이
명시한 대로 **"아직 안 쟀다"는 표시**였고, 08-13 에 라이다를 장착·실측하면서
값이 존재하게 됐다. 표시를 그대로 두고 R5 를 돌리면 스캔이 바퀴축 높이에
꽂혀 지도가 조용히 틀린다.

  origin xyz  "0 0 0" -> "0 0 0.779"      (= 832 스캔평면 - 53 축높이, 단위 mm->m)

🔴 동결 예외 **5회차** (2026-08-02 §10.4 이후 12일 만). 사용자 명시 승인,
범위 = 그 한 줄 + 그 변경이 거짓으로 만든 주석. 기록·전제조건·재개방 조건
3종 = `FREEZE_MANIFEST §10.26`. XML 기능 변경은 origin 한 줄뿐이고
`git diff --stat` 이 1 파일임을 커밋 전에 확인했다.

굽기 당일 **줄자를 다시 쟀다 — 832 mm 로 08-13 과 일치**. 08-13 하루를 줄자
오독 위에서 잃었기 때문에(핸드오프 함정 ①) 값을 물려받지 않고 재측정했다.

🔴 빼는 값은 `0.053`(기하 실측)이지 `0.05698`(역산 계수)이 아니다. `base_joint`
를 이번 묶음에서 안 건드리므로 두 값이 같은 눈금 위에 있어 상쇄되고, 바닥
기준 스캔 평면은 832 로 선다. 한쪽만 고치면 라이다가 7.4 mm 뜬다.

전수 열거: `grep -rn "TODO: " src/tunnel_bringup/` 로 **같은 사실이 2 자리**
(joint 옆 주석 + 파일 머리 미실측 목록)임을 확인하고 둘 다 닫았다. 같은 grep
에 걸린 런치 2건("포트를 udev 링크로 교체")은 **다른 부류라 열지 않았다** —
`99-rplidar.rules` 가 포트를 소스에 안 박고 인자로 넘기기로 한 자리다.

검증: doc_check rc=0 (pytest 184 passed / colcon 247) · XML 파싱 OK ·
몸통 최상면 +155mm 여유 · 08-13 관측 벽 1m 앞 /scan 최소 1.0035m (유령 0건).
⚠ doc_check 초록은 문서 정합이지 사실 증명이 아니다 — 사실은 줄자와
`tf2_echo base_link lidar_link` 가 판정한다.

Caught-by: AGENTS §3-10
  전수 grep 이 파일 머리 45행의 같은 TODO 를 잡았다. joint 옆만 고쳤으면
  파일 머리가 계속 "미실측"이라고 말했을 것이다.

Co-Authored-By: Claude Opus 5 <noreply@anthropic.com>
Claude-Session: https://claude.ai/code/session_01Xg3Sna3zEsMDWbf3vbbLo5

File: src/tunnel_bringup/urdf/robot_real.urdf (robot description, URDF)
Before this commit: robot tunnel_robot_real, 6 links, 5 joints
Joints:
- joint lidar_joint: origin xyz=0 0 0 rpy=0 0 0 -> xyz=0 0 0.779 rpy=0 0 0
